File: LED-Electroscope/LED-Electroscope.kicad_pcb (KiCad board)
At the start: 2 copper layers, 100 x 6 mm, 9 parts, among them J1 Conn_01x01_Female, Q1 2SC1815, Q2 2SA1015

Commit message: fix #1, add description
fix #1, add description
Parts:
- added L1: Logo, teTra:teTra-logo, B.Cu at (185.2, 104.8)
Other:
- board text added: "<< DANGER << << AC (HOT) <<"
- board text added: "LED-Electroscope 211029 V1.0.1"
